File: kicad/release/other-m68k-cpld2.kicad_sch (KiCad schematic)
At the start: 39 parts, among them J3 PS/2, J4 microSD DM3AT-SF-PEJM5, J6 3.5mm audio, SW2 NMI, U7 ATF1508AS-7JX84 (I/O)

Commit message: KiCad rev C1: native 4-bit SD bus (CLK, CMD, DAT0..3 straight from CPLD2 with 10 k pull-ups to 3.3 V, the three 1.8k/3.3k dividers removed, DAT1/DAT2 on CPLD2 pins 16/58), UIO0..3 removed from J8 (pins 5/7/9/11 n/c); ERC 0, DRC 0, rerouted (22 passes, 0 unrouted, 5146 segments, 530 vias); fab package and release snapshot regenerated; ORDER.md notes rev C1 vs the ordered B4
Co-Authored-By: Claude Fable 5.1 <noreply@anthropic.com>
Claude-Session: https://claude.ai/code/session_019bbFLKMxhKXGW6aABP44Z1
Parts:
- removed R24: 3.3k, Resistor_SMD:R_0603_1608Metric, symbol Device:R
- removed R25, R26, R27, R29, R43: 10k, Resistor_SMD:R_0603_1608Metric, symbol Device:R
- removed R28: 1k, Resistor_SMD:R_0603_1608Metric, symbol Device:R
- removed R30: 2.2k, Resistor_SMD:R_0603_1608Metric, symbol Device:R
- added R15, R16, R17, R18, R36: 10k, Resistor_SMD:R_0603_1608Metric, symbol Device:R
- R19: value 1.8k -> 10k; Desc 1.8 k 1% 0603 -> 10 k 1% 0603; LCSC (none) -> C25804; MPN RC0603FR-071K8L -> RC0603FR-0710KL
- R20: value 3.3k -> 10k; Desc 3.3 k 1% 0603 -> 10 k 1% 0603; LCSC C22978 -> C25804; MPN RC0603FR-073K3L -> RC0603FR-0710KL
- R21: value 1.8k -> 1k; Desc 1.8 k 1% 0603 -> 1 k 1% 0603; LCSC (none) -> C21190; MPN RC0603FR-071K8L -> RC0603FR-071KL; PcbNear J4 -> J6
- R22: value 3.3k -> 10k; Desc 3.3 k 1% 0603 -> 10 k 1% 0603; LCSC C22978 -> C25804; MPN RC0603FR-073K3L -> RC0603FR-0710KL; PcbNear J4 -> J6
- R23: value 1.8k -> 2.2k; Desc 1.8 k 1% 0603 -> 2.2 k 1% 0603; LCSC (none) -> C4190; MPN RC0603FR-071K8L -> RC0603FR-072K2L; PcbNear J4 -> J6
Connections:
- net +3V3: now also R19.1, R20.1, R15.1, R16.1, R17.1, R18.1
- net AUDIO: now also R21.1
- net AUDIO_DIV: now also R22.2, R23.1
- net AUDIO_LP: now also R21.2, R22.1
- net GND: now also R23.2, R36.2; no longer R20.2, R22.2
- net PALJMP: now also R36.1
- net SD_CLK: now also J4.5 (CLK), R16.2; no longer R21.1
- net SD_DAT1: now also R19.2, U7.16 (I/O)
- net SD_DAT2: now also R20.2, U7.58 (I/O)
- removed net SD_CLK_3V3: J4.5 (CLK), R21.2, R22.1
- net SD_CS renamed SD_DAT3
- net SD_DAT3: now also J4.2 (DAT3/CD), R15.2; no longer R19.1
- removed net SD_CS_3V3: J4.2 (DAT3/CD), R19.2, R20.1
- net SD_MISO renamed SD_DAT0
- net SD_DAT0: now also R18.2
- net SD_MOSI renamed SD_CMD
- net SD_CMD: now also J4.3 (CMD), R17.2; no longer R23.1
- removed net SD_MOSI_3V3: J4.3 (CMD), R23.2
- net UIO0: no longer names the net of U7.77 (I/O)
- net UIO1: no longer names the net of U7.76 (I/O)
- net UIO2: no longer names the net of U7.75 (I/O)
- net UIO3: no longer names the net of U7.74 (I/O)
- no-connect marks 8 -> 10
Other:
- moved on the sheet: D3, D4, R19, R20, R21, R22, R23, R8, R9, SW2

Commit message: rev C1: audio low-pass 33 nF (C31); sys_read may fill a held BIOS audio buffer
Board: the 1 k / 10 nF low-pass (16 kHz corner, which passed the PDM sigma-delta hiss above
8 kHz) becomes 1 k / 33 nF (4.8 kHz). Same 0603 footprint and nets, so the routed board is
unchanged except C31's value: fab package and release snapshot regenerated from it (DRC 0,
0 unrouted). parts.json: Samsung CL10B333KB8NFNC, LCSC C307488. In the emulator
reconstruction of the tune example the power above 8 kHz relative to the music band drops
from -14 dB to -20.5 dB. ORDER.md names the B4 hand change.

Firmware (spec rev 8 wording): sys_read accepts a destination inside the BIOS audio buffers
while a stream is open (audio_buf_range_ok), so a file streams straight into the buffer the
program holds; sdplay reads raw PDM that way instead of copying. Host tests 401.

Co-Authored-By: Claude Fable 5.1 <noreply@anthropic.com>
Claude-Session: https://claude.ai/code/session_019bbFLKMxhKXGW6aABP44Z1
Parts:
- C31: value 10nF -> 33nF; Desc 10 nF 50 V X7R 0603 -> 33 nF 50 V X7R 0603; LCSC C57112 -> C307488; MPN CL10B103KB8NNNC -> CL10B333KB8NFNC
Changed lines of the file:
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@@
 			)
 		)
-		(property "Value" "10nF"
+		(property "Value" "33nF"
 			(at 111.125 210.82 0)
 			(effects
@@
 			)
 		)
-		(property "MPN" "CL10B103KB8NNNC"
+		(property "MPN" "CL10B333KB8NFNC"
 			(at 110.49 208.28 0)
 			(effects
@@
 			)
 		)
-		(property "LCSC" "C57112"
+		(property "LCSC" "C307488"
 			(at 110.49 208.28 0)
 			(effects
@@
 			)
 		)
-		(property "Desc" "10 nF 50 V X7R 0603"
+		(property "Desc" "33 nF 50 V X7R 0603"
 			(at 110.49 208.28 0)
 			(effects

Commit message: board rev C2 (spec rev 10): front and back edges, S-video jack, serial B header, dedication silkscreen
The rev B4 order was stopped; rev C2 is what goes to PCBWay. The sheet's bottom edge is the
machine's front: J3 PS/2, J6 audio, J4 microSD (LDO behind it), then SW1 RESET and SW2 NMI
with the LEDs D5 PWR, D3 LED0, D4 LED1 behind them, all labelled. The top edge is the back:
J1 USB-C, J2 serial A, J11 serial B (a second FTDI-pinout header on DUART channel B; it
replaces the 2x8 expansion header J8, which carried only channel B and the rails after spec
rev 7), J5 composite, J10 S-video (CUI MD-40SM mini-DIN 4 on the AD724's LUMA and CRMA
outputs through 220 uF and 75 ohm each; new footprint and symbol in kicad/lib). J9 (logic
analyzer) and J7 (JTAG) stand on the left edge with the six series arrays hand-placed in a
spaced column (the auto-placed cluster left one connection unroutable). The flash chips
stand vertically at the right edge; the AD724 section sits right of the S-video jack; the
bus buffers moved under the SRAMs. The open area under the CPU carries "Griffin Jr.",
"October 2026", "I love you, Kris!" and the revision; connector labels are placed where
the silkscreen checker finds them free of pads and other silk.

Routed by freerouting (optimizer on): 0 DRC violations, 0 unrouted. Fab package and
release regenerated; ORDER.md rewritten for rev C2. Spec rev 10 carries only the connector
wording (serial headers, S-video); no register or firmware change.

Co-Authored-By: Claude Fable 5.1 <noreply@anthropic.com>
Claude-Session: https://claude.ai/code/session_019bbFLKMxhKXGW6aABP44Z1
Parts:
- D3, D4: PcbNear U7 -> SW2
Changed lines of the file:
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@@
 			)
 		)
-		(property "PcbNear" "U7"
+		(property "PcbNear" "SW2"
 			(at 49.53 317.5 0)
 			(effects
@@
 			)
 		)
-		(property "PcbNear" "U7"
-			(at 302.26 289.56 0)
-			(effects
+		(property "PcbNear" "SW2"
+			(at 302.26 289.56 0)
+			(effects

Commit message: rev C3 BOM: in-stock substitutes from the PCBWay quote: ECS-2200B-240 oscillator, Assmann PLCC-84 and DIP-40 sockets, generic DIP-64 socket acceptable
Co-Authored-By: Claude Fable 5.1 <noreply@anthropic.com>
Claude-Session: https://claude.ai/code/session_019bbFLKMxhKXGW6aABP44Z1
Parts:
- U7: Socket_Desc PLCC-84 through-hole socket, 1.27 mm pitch (RS 7019411) -> PLCC-84 through-hole socket, 1.27 mm pitch (DigiKey 5023770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; Socket_MPN 540-88-084-24-008 -> A-CCS-084-Z-T; Socket_Manufacturer Preci-dip -> Assmann WSW
Changed lines of the file:
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@@
 			)
 		)
-		(property "Socket_Manufacturer" "Preci-dip"
+		(property "Socket_Manufacturer" "Assmann WSW"
 			(at 62.23 76.2 0)
 			(effects
@@
 			)
 		)
-		(property "Socket_MPN" "540-88-084-24-008"
+		(property "Socket_MPN" "A-CCS-084-Z-T"
 			(at 62.23 76.2 0)
 			(effects
@@
 			)
 		)
-		(property "Socket_Desc" "PLCC-84 through-hole socket, 1.27 mm pitch (RS 7019411)"
+		(property "Socket_Desc" "PLCC-84 through-hole socket, 1.27 mm pitch (DigiKey 5023770 / AE11110-ND, RS 674-2555; any THT PLCC-84 socket with the JEDEC pin pattern is acceptable)"
 			(at 62.23 76.2 0)
 			(effects

Commit message: BOM: PCBWay descriptions carry only the part and its substitution rule; our sourcing remarks move to a Note field in parts.json, the KiCad BOM and the customer-parts list
Co-Authored-By: Claude Fable 5.1 <noreply@anthropic.com>
Claude-Session: https://claude.ai/code/session_019bbFLKMxhKXGW6aABP44Z1
Parts:
- U7: Socket_Desc PLCC-84 through-hole socket, 1.27 mm pitch (DigiKey 5023770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 -> PLCC-84 through-hole socket, 1.27 mm pitch; any THT PLCC-84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; Socket_Note (none) -> DigiKey 5023770 / AE11110-ND, RS 674-2555. Replaces the Pre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
Changed lines of the file:
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@@
 			)
 		)
-		(property "Socket_Desc" "PLCC-84 through-hole socket, 1.27 mm pitch (DigiKey 5023770 / AE11110-ND, RS 674-2555; any THT PLCC-84 socket with the JEDEC pin pattern is acceptable)"
+		(property "Socket_Desc" "PLCC-84 through-hole socket, 1.27 mm pitch; any THT PLCC-84 socket with the JEDEC pin pattern is acceptable"
 			(at 62.23 76.2 0)
 			(effects
+				(font
+					(size 1.27 1.27)
+				)
+				(hide yes)
+			)
+		)
+		(property "Socket_Note" "DigiKey 5023770 / AE11110-ND, RS 674-2555. Replaces the Preci-dip PCBWay could not source (2026-10)"
+			(at 62.23 76.2 0)
+			(effects
