File: kicad/release/other-m68k-memory.kicad_sch (KiCad schematic)
At the start: 12 parts, among them U2 AS6C4008-55PCN (upper, D15..D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, U3 AS6C4008-55PCN (lower, D7..D0), U4 SST39SF040-70 (even, D15..D8), U5 SST39SF040-70 (odd, D7..D0), U8 74AHCT245 (hi), U9 74AHCT245 (lo)

Commit message: rev C3 BOM: the SRAM, flash and AD724 leave the assembly BOM (we buy and fit them); ORDER.md gets the order-form substitution note
PCBWay quoted $281 of parts for the B4 bill, $170 of it the five chips (AD724 $77,
two AS6C4008 $31, two SST39SF040 $9.76) plus $60 for two machined sockets. The chips
are now Assembly=customer / Chip_Supply=customer: the sockets ship empty, U11 is
hand-soldered here, and nothing is consigned. ORDER.md gains the socket and substitute
wording for the order form and the list of connectors to keep on the named part.

Co-Authored-By: Claude Fable 5.1 <noreply@anthropic.com>
Claude-Session: https://claude.ai/code/session_019bbFLKMxhKXGW6aABP44Z1
Parts:
- U2, U3, U4, U5: Chip_Supply pcba -> customer
Changed lines of the file:
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@@
 			)
 		)
-		(property "Chip_Supply" "pcba"
+		(property "Chip_Supply" "customer"
 			(at 151.13 62.23 0)
 			(effects
@@
 			)
 		)
-		(property "Chip_Supply" "pcba"
+		(property "Chip_Supply" "customer"
 			(at 59.69 62.23 0)
 			(effects
@@
 			)
 		)
-		(property "Chip_Supply" "pcba"
+		(property "Chip_Supply" "customer"
 			(at 57.15 143.51 0)
 			(effects
@@
 			)
 		)
-		(property "Chip_Supply" "pcba"
-			(at 238.76 53.34 0)
-			(effects
+		(property "Chip_Supply" "customer"
+			(at 238.76 53.34 0)
+			(effects

Commit message: BOM: PCBWay descriptions carry only the part and its substitution rule; our sourcing remarks move to a Note field in parts.json, the KiCad BOM and the customer-parts list
Co-Authored-By: Claude Fable 5.1 <noreply@anthropic.com>
Claude-Session: https://claude.ai/code/session_019bbFLKMxhKXGW6aABP44Z1
Parts:
- U2, U3, U4, U5: Socket_Desc DIP-32 socket, 15.24 mm rows, stamped dual-wipe tin contact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 -> DIP-32 socket, 15.24 mm rows, stamped dual-wipe tin contacts; Socket_Note (none) -> RS 674-2463; A 32-LC-TR is the same socket at DigiKey
Changed lines of the file:
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@@
 			)
 		)
-		(property "Socket_Desc" "DIP-32 socket, 15.24 mm rows, stamped dual-wipe tin contacts (RS 674-2463; A 32-LC-TR is the same socket at DigiKey)"
+		(property "Socket_Desc" "DIP-32 socket, 15.24 mm rows, stamped dual-wipe tin contacts"
+			(at 151.13 62.23 0)
+			(effects
+				(font
+					(size 1.27 1.27)
+				)
+				(hide yes)
+			)
+		)
+		(property "Socket_Note" "RS 674-2463; A 32-LC-TR is the same socket at DigiKey"
 			(at 151.13 62.23 0)
 			(effects
@@
 			)
 		)
-		(property "Socket_Desc" "DIP-32 socket, 15.24 mm rows, stamped dual-wipe tin contacts (RS 674-2463; A 32-LC-TR is the same socket at DigiKey)"
+		(property "Socket_Desc" "DIP-32 socket, 15.24 mm rows, stamped dual-wipe tin contacts"
+			(at 59.69 62.23 0)
+			(effects
+				(font
+					(size 1.27 1.27)
+				)
+				(hide yes)
+			)
+		)
+		(property "Socket_Note" "RS 674-2463; A 32-LC-TR is the same socket at DigiKey"
 			(at 59.69 62.23 0)
 			(effects
@@
 			)
 		)
-		(property "Socket_Desc" "DIP-32 socket, 15.24 mm rows, stamped dual-wipe tin contacts (RS 674-2463; A 32-LC-TR is the same socket at DigiKey)"
+		(property "Socket_Desc" "DIP-32 socket, 15.24 mm rows, stamped dual-wipe tin contacts"
+			(at 57.15 143.51 0)
+			(effects
+				(font
+					(size 1.27 1.27)
+				)
+				(hide yes)
+			)
+		)
+		(property "Socket_Note" "RS 674-2463; A 32-LC-TR is the same socket at DigiKey"
 			(at 57.15 143.51 0)
 			(effects
@@
 			)
 		)
-		(property "Socket_Desc" "DIP-32 socket, 15.24 mm rows, stamped dual-wipe tin contacts (RS 674-2463; A 32-LC-TR is the same socket at DigiKey)"
-			(at 238.76 53.34 0)
-			(effects
+		(property "Socket_Desc" "DIP-32 socket, 15.24 mm rows, stamped dual-wipe tin contacts"
+			(at 238.76 53.34 0)
+			(effects
+				(font
+					(size 1.27 1.27)
+				)
+				(hide yes)
+			)
+		)
+		(property "Socket_Note" "RS 674-2463; A 32-LC-TR is the same socket at DigiKey"
+			(at 238.76 53.34 0)
+			(effects
