File: kicad/release/other-m68k-power.kicad_sch (KiCad schematic)
At the start: 19 parts, among them J1 USB-C power, U12 AP2112K-3.3

Commit message: KiCad rev C1: native 4-bit SD bus (CLK, CMD, DAT0..3 straight from CPLD2 with 10 k pull-ups to 3.3 V, the three 1.8k/3.3k dividers removed, DAT1/DAT2 on CPLD2 pins 16/58), UIO0..3 removed from J8 (pins 5/7/9/11 n/c); ERC 0, DRC 0, rerouted (22 passes, 0 unrouted, 5146 segments, 530 vias); fab package and release snapshot regenerated; ORDER.md notes rev C1 vs the ordered B4
Co-Authored-By: Claude Fable 5.1 <noreply@anthropic.com>
Claude-Session: https://claude.ai/code/session_019bbFLKMxhKXGW6aABP44Z1
Parts:
- removed R54, R55: 5.1k, Resistor_SMD:R_0603_1608Metric, symbol Device:R
- removed R56: 1k, Resistor_SMD:R_0603_1608Metric, symbol Device:R
- added R47, R48: 5.1k, Resistor_SMD:R_0603_1608Metric, symbol Device:R
- added R49: 1k, Resistor_SMD:R_0603_1608Metric, symbol Device:R
Connections:
- net CC1: now also R47.1
- net CC2: now also R48.1
- net GND: now also R47.2, R48.2
- net PWRLED_A: now also R49.2
- net VCC: now also R49.1
Changed lines of the file:
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@@
 	(title_block
 		(title "power")
-		(rev "A")
+		(rev "C1")
 		(comment 1 "generated by kicad/gen_sch.py - do not edit")
 	)
@@
 		(on_board yes)
 		(dnp no)
-		(property "Reference" "R56"
+		(property "Reference" "R49"
 			(at 174.752 139.7 90)
 			(effects
@@
 			(project "other-m68k"
 				(path "/0bd472a6-02e9-5c95-a886-c7baf9734bb2/31d43ba6-5b87-5475-9f10-ec280f14fb9b"
-					(reference "R56")
+					(reference "R49")
 					(unit 1)
 				)
@@
 		(on_board yes)
 		(dnp no)
-		(property "Reference" "R55"
+		(property "Reference" "R48"
 			(at 111.252 139.7 90)
 			(effects
@@
 			(project "other-m68k"
 				(path "/0bd472a6-02e9-5c95-a886-c7baf9734bb2/31d43ba6-5b87-5475-9f10-ec280f14fb9b"
-					(reference "R55")
+					(reference "R48")
 					(unit 1)
 				)
@@
 		(on_board yes)
 		(dnp no)
-		(property "Reference" "R54"
+		(property "Reference" "R47"
 			(at 47.752 139.7 90)
 			(effects
@@
 			(project "other-m68k"
 				(path "/0bd472a6-02e9-5c95-a886-c7baf9734bb2/31d43ba6-5b87-5475-9f10-ec280f14fb9b"
-					(reference "R54")
+					(reference "R47")
 					(unit 1)
 				)
@@
 		(on_board no)
 		(dnp no)
-		(property "Reference" "#PWR146"
+		(property "Reference" "#PWR142"
 			(at 138.43 48.26 0)
 			(effects
@@
 			(project "other-m68k"
 				(path "/0bd472a6-02e9-5c95-a886-c7baf9734bb2/31d43ba6-5b87-5475-9f10-ec280f14fb9b"
-					(reference "#PWR146")
+					(reference "#PWR142")
 					(unit 1)
 				)
@@
 		(on_board no)
 		(dnp no)
-		(property "Reference" "#PWR147"
+		(property "Reference" "#PWR143"
 			(at 46.99 69.85 0)
 			(effects
@@
 			(project "other-m68k"
 				(path "/0bd472a6-02e9-5c95-a886-c7baf9734bb2/31d43ba6-5b87-5475-9f10-ec280f14fb9b"
-					(reference "#PWR147")
+					(reference "#PWR143")
 					(unit 1)
 				)
@@
 		(on_board no)
 		(dnp no)
-		(property "Reference" "#PWR148"
+		(property "Reference" "#PWR144"
 			(at 54.61 69.85 0)
 			(effects
@@
 			(project "other-m68k"
 				(path "/0bd472a6-02e9-5c95-a886-c7baf9734bb2/31d43ba6-5b87-5475-9f10-ec280f14fb9b"
-					(reference "#PWR148")
+					(reference "#PWR144")
 					(unit 1)
 				)
@@
 		(on_board no)
 		(dnp no)
-		(property "Reference" "#PWR149"
+		(property "Reference" "#PWR145"
 			(at 234.95 78.74 0)
 			(effects
@@
 			(project "other-m68k"
 				(path "/0bd472a6-02e9-5c95-a886-c7baf9734bb2/31d43ba6-5b87-5475-9f10-ec280f14fb9b"
-					(reference "#PWR149")
+					(reference "#PWR145")
 					(unit 1)
 				)
@@
 		(on_board no)
 		(dnp no)
-		(property "Reference" "#PWR150"
+		(property "Reference" "#PWR146"
 			(at 207.01 44.45 0)
 			(effects
@@
 			(project "other-m68k"
 				(path "/0bd472a6-02e9-5c95-a886-c7baf9734bb2/31d43ba6-5b87-5475-9f10-ec280f14fb9b"
-					(reference "#PWR150")
+					(reference "#PWR146")
 					(unit 1)
 				)
@@
 		(on_board no)
 		(dnp no)
-		(property "Reference" "#PWR151"
+		(property "Reference" "#PWR147"
 			(at 45.72 97.79 0)
 			(effects
@@
 			(project "other-m68k"
 				(path "/0bd472a6-02e9-5c95-a886-c7baf9734bb2/31d43ba6-5b87-5475-9f10-ec280f14fb9b"
-					(reference "#PWR151")
+					(reference "#PWR147")
 					(unit 1)
 				)
@@
 		(on_board no)
 		(dnp no)
-		(property "Reference" "#PWR152"
+		(property "Reference" "#PWR148"
 			(at 109.22 97.79 0)
 			(effects
@@
 			(project "other-m68k"
 				(path "/0bd472a6-02e9-5c95-a886-c7baf9734bb2/31d43ba6-5b87-5475-9f10-ec280f14fb9b"
-					(reference "#PWR152")
+					(reference "#PWR148")
 					(unit 1)
 				)
@@
 		(on_board no)
 		(dnp no)
-		(property "Reference" "#PWR153"
+		(property "Reference" "#PWR149"
 			(at 171.45 97.79 0)
 			(effects
@@
 			(project "other-m68k"
 				(path "/0bd472a6-02e9-5c95-a886-c7baf9734bb2/31d43ba6-5b87-5475-9f10-ec280f14fb9b"
-					(reference "#PWR153")
+					(reference "#PWR149")
 					(unit 1)
 				)
@@
 		(on_board no)
 		(dnp no)
-		(property "Reference" "#PWR154"
+		(property "Reference" "#PWR150"
 			(at 45.72 153.67 0)
 			(effects
@@
 			(project "other-m68k"
 				(path "/0bd472a6-02e9-5c95-a886-c7baf9734bb2/31d43ba6-5b87-5475-9f10-ec280f14fb9b"
-					(reference "#PWR154")
+					(reference "#PWR150")
 					(unit 1)
 				)
@@
 		(on_board no)
 		(dnp no)
-		(property "Reference" "#PWR155"
+		(property "Reference" "#PWR151"
 			(at 109.22 153.67 0)
 			(effects
@@
 			(project "other-m68k"
 				(path "/0bd472a6-02e9-5c95-a886-c7baf9734bb2/31d43ba6-5b87-5475-9f10-ec280f14fb9b"
-					(reference "#PWR155")
+					(reference "#PWR151")
 					(unit 1)
 				)
@@
 		(on_board no)
 		(dnp no)
-		(property "Reference" "#PWR156"
+		(property "Reference" "#PWR152"
 			(at 46.99 107.95 0)
 			(effects
@@
 			(project "other-m68k"
 				(path "/0bd472a6-02e9-5c95-a886-c7baf9734bb2/31d43ba6-5b87-5475-9f10-ec280f14fb9b"
-					(reference "#PWR156")
+					(reference "#PWR152")
 					(unit 1)
 				)
@@
 		(on_board no)
 		(dnp no)
-		(property "Reference" "#PWR157"
+		(property "Reference" "#PWR153"
 			(at 46.99 125.73 0)
 			(effects
@@
 			(project "other-m68k"
 				(path "/0bd472a6-02e9-5c95-a886-c7baf9734bb2/31d43ba6-5b87-5475-9f10-ec280f14fb9b"
-					(reference "#PWR157")
+					(reference "#PWR153")
 					(unit 1)
 				)
@@
 		(on_board no)
 		(dnp no)
-		(property "Reference" "#PWR158"
+		(property "Reference" "#PWR154"
 			(at 111.76 107.95 0)
 			(effects
@@
 			(project "other-m68k"
 				(path "/0bd472a6-02e9-5c95-a886-c7baf9734bb2/31d43ba6-5b87-5475-9f10-ec280f14fb9b"
-					(reference "#PWR158")
+					(reference "#PWR154")
 					(unit 1)
 				)
@@
 		(on_board no)
 		(dnp no)
-		(property "Reference" "#PWR159"
+		(property "Reference" "#PWR155"
 			(at 111.76 125.73 0)
 			(effects
@@
 			(project "other-m68k"
 				(path "/0bd472a6-02e9-5c95-a886-c7baf9734bb2/31d43ba6-5b87-5475-9f10-ec280f14fb9b"
-					(reference "#PWR159")
+					(reference "#PWR155")
 					(unit 1)
 				)
@@
 		(on_board no)
 		(dnp no)
-		(property "Reference" "#PWR160"
+		(property "Reference" "#PWR156"
 			(at 172.72 135.89 0)
 			(effects
@@
 			(project "other-m68k"
 				(path "/0bd472a6-02e9-5c95-a886-c7baf9734bb2/31d43ba6-5b87-5475-9f10-ec280f14fb9b"
-					(reference "#PWR160")
+					(reference "#PWR156")
 					(unit 1)
 				)
@@
 		(on_board no)
 		(dnp no)
-		(property "Reference" "#PWR161"
+		(property "Reference" "#PWR157"
 			(at 175.26 107.95 0)
 			(effects
@@
 			(project "other-m68k"
 				(path "/0bd472a6-02e9-5c95-a886-c7baf9734bb2/31d43ba6-5b87-5475-9f10-ec280f14fb9b"
-					(reference "#PWR161")
+					(reference "#PWR157")
 					(unit 1)
 				)
@@
 		(on_board no)
 		(dnp no)
-		(property "Reference" "#PWR162"
+		(property "Reference" "#PWR158"
 			(at 175.26 125.73 0)
 			(effects
@@
 			(project "other-m68k"
 				(path "/0bd472a6-02e9-5c95-a886-c7baf9734bb2/31d43ba6-5b87-5475-9f10-ec280f14fb9b"
-					(reference "#PWR162")
+					(reference "#PWR158")
 					(unit 1)
 				)
@@
 		(on_board no)
 		(dnp no)
-		(property "Reference" "#PWR163"
+		(property "Reference" "#PWR159"
 			(at 240.03 107.95 0)
 			(effects
@@
 			(project "other-m68k"
 				(path "/0bd472a6-02e9-5c95-a886-c7baf9734bb2/31d43ba6-5b87-5475-9f10-ec280f14fb9b"
-					(reference "#PWR163")
+					(reference "#PWR159")
 					(unit 1)
 				)
@@
 		(on_board no)
 		(dnp no)
-		(property "Reference" "#PWR164"
+		(property "Reference" "#PWR160"
 			(at 240.03 125.73 0)
 			(effects
@@
 			(project "other-m68k"
 				(path "/0bd472a6-02e9-5c95-a886-c7baf9734bb2/31d43ba6-5b87-5475-9f10-ec280f14fb9b"
-					(reference "#PWR164")
+					(reference "#PWR160")
 					(unit 1)
 				)
@@
 		(on_board no)
 		(dnp no)
-		(property "Reference" "#PWR165"
+		(property "Reference" "#PWR161"
 			(at 168.91 180.34 0)
 			(effects
@@
 			(project "other-m68k"
 				(path "/0bd472a6-02e9-5c95-a886-c7baf9734bb2/31d43ba6-5b87-5475-9f10-ec280f14fb9b"
-					(reference "#PWR165")
+					(reference "#PWR161")
 					(unit 1)
 				)

Commit message: board rev C2 (spec rev 10): front and back edges, S-video jack, serial B header, dedication silkscreen
The rev B4 order was stopped; rev C2 is what goes to PCBWay. The sheet's bottom edge is the
machine's front: J3 PS/2, J6 audio, J4 microSD (LDO behind it), then SW1 RESET and SW2 NMI
with the LEDs D5 PWR, D3 LED0, D4 LED1 behind them, all labelled. The top edge is the back:
J1 USB-C, J2 serial A, J11 serial B (a second FTDI-pinout header on DUART channel B; it
replaces the 2x8 expansion header J8, which carried only channel B and the rails after spec
rev 7), J5 composite, J10 S-video (CUI MD-40SM mini-DIN 4 on the AD724's LUMA and CRMA
outputs through 220 uF and 75 ohm each; new footprint and symbol in kicad/lib). J9 (logic
analyzer) and J7 (JTAG) stand on the left edge with the six series arrays hand-placed in a
spaced column (the auto-placed cluster left one connection unroutable). The flash chips
stand vertically at the right edge; the AD724 section sits right of the S-video jack; the
bus buffers moved under the SRAMs. The open area under the CPU carries "Griffin Jr.",
"October 2026", "I love you, Kris!" and the revision; connector labels are placed where
the silkscreen checker finds them free of pads and other silk.

Routed by freerouting (optimizer on): 0 DRC violations, 0 unrouted. Fab package and
release regenerated; ORDER.md rewritten for rev C2. Spec rev 10 carries only the connector
wording (serial headers, S-video); no register or firmware change.

Co-Authored-By: Claude Fable 5.1 <noreply@anthropic.com>
Claude-Session: https://claude.ai/code/session_019bbFLKMxhKXGW6aABP44Z1
Parts:
- removed C46: 100uF, Capacitor_THT:CP_Radial_D6.3mm_P2.50mm, symbol Device:C_Polarized
- removed C47: 10uF, Capacitor_SMD:C_0805_2012Metric, symbol Device:C
- removed R47, R48: 5.1k, Resistor_SMD:R_0603_1608Metric, symbol Device:R
- added C50, C51: 1uF, Capacitor_SMD:C_0603_1608Metric, symbol Device:C
- added R50: 5.1k, Resistor_SMD:R_0603_1608Metric, symbol Device:R
- added R51: 1k, Resistor_SMD:R_0603_1608Metric, symbol Device:R
- C48: value 1uF -> 100uF; footprint Capacitor_SMD:C_0603_1608Metric -> Capacitor_THT:CP_Radial_D6.3mm_P2.50mm; symbol Device:C -> Device:C_Polarized; Desc 1 uF 50 V X5R 0603 -> 100 uF 35 V electrolytic, 6.3 mm dia, 2.5 mm pitch (the 16 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; LCSC C15849 -> (none); MPN CL10A105KB8NNNC -> 35ZLH100MEFC6.3X11; Manufacturer Samsung -> Rubycon; PcbNear U12 -> J1
- C49: value 1uF -> 10uF; footprint Capacitor_SMD:C_0603_1608Metric -> Capacitor_SMD:C_0805_2012Metric; Desc 1 uF 50 V X5R 0603 -> 10 uF 25 V X5R 0805; LCSC C15849 -> C15850; MPN CL10A105KB8NNNC -> CL21A106KAYNNNE; PcbNear U12 -> J1
- D5: PcbNear J1 -> SW1
- R49: value 1k -> 5.1k; Desc 1 k 1% 0603 -> 5.1 k 1% 0603 (USB-C CC pull-downs); LCSC C21190 -> C23186; MPN RC0603FR-071KL -> RC0603FR-075K1L
Connections:
- net +3V3: now also C51.1; no longer C49.1
- net CC1: now also R49.1
- net CC2: now also R50.1
- net GND: now also R49.2, C50.2, C51.2, R50.2
- net PWRLED_A: now also R51.2; no longer R49.2
- net VCC: now also C49.1, C50.1, R51.1; no longer R49.1
Other:
- moved on the sheet: C49, R49
Changed lines of the file:
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@@
 		(on_board yes)
 		(dnp no)
-		(property "Reference" "C49"
+		(property "Reference" "C51"
 			(at 240.665 109.22 0)
 			(effects
@@
 			(project "other-m68k"
 				(path "/0bd472a6-02e9-5c95-a886-c7baf9734bb2/31d43ba6-5b87-5475-9f10-ec280f14fb9b"
-					(reference "C49")
+					(reference "C51")
 					(unit 1)
 				)
@@
 		(on_board yes)
 		(dnp no)
-		(property "Reference" "C48"
+		(property "Reference" "C50"
 			(at 175.895 109.22 0)
 			(effects
@@
 			(project "other-m68k"
 				(path "/0bd472a6-02e9-5c95-a886-c7baf9734bb2/31d43ba6-5b87-5475-9f10-ec280f14fb9b"
-					(reference "C48")
+					(reference "C50")
 					(unit 1)
 				)
@@
 			)
 		)
-		(property "PcbNear" "J1"
+		(property "PcbNear" "SW1"
 			(at 233.68 166.37 0)
 			(effects
@@
 		(on_board yes)
 		(dnp no)
-		(property "Reference" "R49"
+		(property "Reference" "R51"
 			(at 174.752 139.7 90)
 			(effects
@@
 			(project "other-m68k"
 				(path "/0bd472a6-02e9-5c95-a886-c7baf9734bb2/31d43ba6-5b87-5475-9f10-ec280f14fb9b"
-					(reference "R49")
+					(reference "R51")
 					(unit 1)
 				)
@@
 		(on_board yes)
 		(dnp no)
-		(property "Reference" "C47"
+		(property "Reference" "C49"
 			(at 112.395 109.22 0)
 			(effects
@@
 			(project "other-m68k"
 				(path "/0bd472a6-02e9-5c95-a886-c7baf9734bb2/31d43ba6-5b87-5475-9f10-ec280f14fb9b"
-					(reference "C47")
+					(reference "C49")
 					(unit 1)
 				)
@@
 		(on_board yes)
 		(dnp no)
-		(property "Reference" "C46"
+		(property "Reference" "C48"
 			(at 47.625 109.22 0)
 			(effects
@@
 			(project "other-m68k"
 				(path "/0bd472a6-02e9-5c95-a886-c7baf9734bb2/31d43ba6-5b87-5475-9f10-ec280f14fb9b"
-					(reference "C46")
+					(reference "C48")
 					(unit 1)
 				)
@@
 		(on_board yes)
 		(dnp no)
-		(property "Reference" "R48"
+		(property "Reference" "R50"
 			(at 111.252 139.7 90)
 			(effects
@@
 			(project "other-m68k"
 				(path "/0bd472a6-02e9-5c95-a886-c7baf9734bb2/31d43ba6-5b87-5475-9f10-ec280f14fb9b"
-					(reference "R48")
+					(reference "R50")
 					(unit 1)
 				)
@@
 		(on_board yes)
 		(dnp no)
-		(property "Reference" "R47"
+		(property "Reference" "R49"
 			(at 47.752 139.7 90)
 			(effects
@@
 			(project "other-m68k"
 				(path "/0bd472a6-02e9-5c95-a886-c7baf9734bb2/31d43ba6-5b87-5475-9f10-ec280f14fb9b"
-					(reference "R47")
+					(reference "R49")
 					(unit 1)
 				)
@@
 		(on_board no)
 		(dnp no)
-		(property "Reference" "#PWR142"
+		(property "Reference" "#PWR143"
 			(at 138.43 48.26 0)
 			(effects
@@
 			(project "other-m68k"
 				(path "/0bd472a6-02e9-5c95-a886-c7baf9734bb2/31d43ba6-5b87-5475-9f10-ec280f14fb9b"
-					(reference "#PWR142")
+					(reference "#PWR143")
 					(unit 1)
 				)
@@
 		(on_board no)
 		(dnp no)
-		(property "Reference" "#PWR143"
+		(property "Reference" "#PWR144"
 			(at 46.99 69.85 0)
 			(effects
@@
 			(project "other-m68k"
 				(path "/0bd472a6-02e9-5c95-a886-c7baf9734bb2/31d43ba6-5b87-5475-9f10-ec280f14fb9b"
-					(reference "#PWR143")
+					(reference "#PWR144")
 					(unit 1)
 				)
@@
 		(on_board no)
 		(dnp no)
-		(property "Reference" "#PWR144"
+		(property "Reference" "#PWR145"
 			(at 54.61 69.85 0)
 			(effects
@@
 			(project "other-m68k"
 				(path "/0bd472a6-02e9-5c95-a886-c7baf9734bb2/31d43ba6-5b87-5475-9f10-ec280f14fb9b"
-					(reference "#PWR144")
+					(reference "#PWR145")
 					(unit 1)
 				)
@@
 		(on_board no)
 		(dnp no)
-		(property "Reference" "#PWR145"
+		(property "Reference" "#PWR146"
 			(at 234.95 78.74 0)
 			(effects
@@
 			(project "other-m68k"
 				(path "/0bd472a6-02e9-5c95-a886-c7baf9734bb2/31d43ba6-5b87-5475-9f10-ec280f14fb9b"
-					(reference "#PWR145")
+					(reference "#PWR146")
 					(unit 1)
 				)
@@
 		(on_board no)
 		(dnp no)
-		(property "Reference" "#PWR146"
+		(property "Reference" "#PWR147"
 			(at 207.01 44.45 0)
 			(effects
@@
 			(project "other-m68k"
 				(path "/0bd472a6-02e9-5c95-a886-c7baf9734bb2/31d43ba6-5b87-5475-9f10-ec280f14fb9b"
-					(reference "#PWR146")
+					(reference "#PWR147")
 					(unit 1)
 				)
@@
 		(on_board no)
 		(dnp no)
-		(property "Reference" "#PWR147"
+		(property "Reference" "#PWR148"
 			(at 45.72 97.79 0)
 			(effects
@@
 			(project "other-m68k"
 				(path "/0bd472a6-02e9-5c95-a886-c7baf9734bb2/31d43ba6-5b87-5475-9f10-ec280f14fb9b"
-					(reference "#PWR147")
+					(reference "#PWR148")
 					(unit 1)
 				)
@@
 		(on_board no)
 		(dnp no)
-		(property "Reference" "#PWR148"
+		(property "Reference" "#PWR149"
 			(at 109.22 97.79 0)
 			(effects
@@
 			(project "other-m68k"
 				(path "/0bd472a6-02e9-5c95-a886-c7baf9734bb2/31d43ba6-5b87-5475-9f10-ec280f14fb9b"
-					(reference "#PWR148")
+					(reference "#PWR149")
 					(unit 1)
 				)
@@
 		(on_board no)
 		(dnp no)
-		(property "Reference" "#PWR149"
+		(property "Reference" "#PWR150"
 			(at 171.45 97.79 0)
 			(effects
@@
 			(project "other-m68k"
 				(path "/0bd472a6-02e9-5c95-a886-c7baf9734bb2/31d43ba6-5b87-5475-9f10-ec280f14fb9b"
-					(reference "#PWR149")
+					(reference "#PWR150")
 					(unit 1)
 				)
@@
 		(on_board no)
 		(dnp no)
-		(property "Reference" "#PWR150"
+		(property "Reference" "#PWR151"
 			(at 45.72 153.67 0)
 			(effects
@@
 			(project "other-m68k"
 				(path "/0bd472a6-02e9-5c95-a886-c7baf9734bb2/31d43ba6-5b87-5475-9f10-ec280f14fb9b"
-					(reference "#PWR150")
+					(reference "#PWR151")
 					(unit 1)
 				)
@@
 		(on_board no)
 		(dnp no)
-		(property "Reference" "#PWR151"
+		(property "Reference" "#PWR152"
 			(at 109.22 153.67 0)
 			(effects
@@
 			(project "other-m68k"
 				(path "/0bd472a6-02e9-5c95-a886-c7baf9734bb2/31d43ba6-5b87-5475-9f10-ec280f14fb9b"
-					(reference "#PWR151")
+					(reference "#PWR152")
 					(unit 1)
 				)
@@
 		(on_board no)
 		(dnp no)
-		(property "Reference" "#PWR152"
+		(property "Reference" "#PWR153"
 			(at 46.99 107.95 0)
 			(effects
@@
 			(project "other-m68k"
 				(path "/0bd472a6-02e9-5c95-a886-c7baf9734bb2/31d43ba6-5b87-5475-9f10-ec280f14fb9b"
-					(reference "#PWR152")
+					(reference "#PWR153")
 					(unit 1)
 				)
@@
 		(on_board no)
 		(dnp no)
-		(property "Reference" "#PWR153"
+		(property "Reference" "#PWR154"
 			(at 46.99 125.73 0)
 			(effects
@@
 			(project "other-m68k"
 				(path "/0bd472a6-02e9-5c95-a886-c7baf9734bb2/31d43ba6-5b87-5475-9f10-ec280f14fb9b"
-					(reference "#PWR153")
+					(reference "#PWR154")
 					(unit 1)
 				)
@@
 		(on_board no)
 		(dnp no)
-		(property "Reference" "#PWR154"
+		(property "Reference" "#PWR155"
 			(at 111.76 107.95 0)
 			(effects
@@
 			(project "other-m68k"
 				(path "/0bd472a6-02e9-5c95-a886-c7baf9734bb2/31d43ba6-5b87-5475-9f10-ec280f14fb9b"
-					(reference "#PWR154")
+					(reference "#PWR155")
 					(unit 1)
 				)
@@
 		(on_board no)
 		(dnp no)
-		(property "Reference" "#PWR155"
+		(property "Reference" "#PWR156"
 			(at 111.76 125.73 0)
 			(effects
@@
 			(project "other-m68k"
 				(path "/0bd472a6-02e9-5c95-a886-c7baf9734bb2/31d43ba6-5b87-5475-9f10-ec280f14fb9b"
-					(reference "#PWR155")
+					(reference "#PWR156")
 					(unit 1)
 				)
@@
 		(on_board no)
 		(dnp no)
-		(property "Reference" "#PWR156"
+		(property "Reference" "#PWR157"
 			(at 172.72 135.89 0)
 			(effects
@@
 			(project "other-m68k"
 				(path "/0bd472a6-02e9-5c95-a886-c7baf9734bb2/31d43ba6-5b87-5475-9f10-ec280f14fb9b"
-					(reference "#PWR156")
+					(reference "#PWR157")
 					(unit 1)
 				)
@@
 		(on_board no)
 		(dnp no)
-		(property "Reference" "#PWR157"
+		(property "Reference" "#PWR158"
 			(at 175.26 107.95 0)
 			(effects
@@
 			(project "other-m68k"
 				(path "/0bd472a6-02e9-5c95-a886-c7baf9734bb2/31d43ba6-5b87-5475-9f10-ec280f14fb9b"
-					(reference "#PWR157")
+					(reference "#PWR158")
 					(unit 1)
 				)
@@
 		(on_board no)
 		(dnp no)
-		(property "Reference" "#PWR158"
+		(property "Reference" "#PWR159"
 			(at 175.26 125.73 0)
 			(effects
@@
 			(project "other-m68k"
 				(path "/0bd472a6-02e9-5c95-a886-c7baf9734bb2/31d43ba6-5b87-5475-9f10-ec280f14fb9b"
-					(reference "#PWR158")
+					(reference "#PWR159")
 					(unit 1)
 				)
@@
 		(on_board no)
 		(dnp no)
-		(property "Reference" "#PWR159"
+		(property "Reference" "#PWR160"
 			(at 240.03 107.95 0)
 			(effects
@@
 			(project "other-m68k"
 				(path "/0bd472a6-02e9-5c95-a886-c7baf9734bb2/31d43ba6-5b87-5475-9f10-ec280f14fb9b"
-					(reference "#PWR159")
+					(reference "#PWR160")
 					(unit 1)
 				)
@@
 		(on_board no)
 		(dnp no)
-		(property "Reference" "#PWR160"
+		(property "Reference" "#PWR161"
 			(at 240.03 125.73 0)
 			(effects
@@
 			(project "other-m68k"
 				(path "/0bd472a6-02e9-5c95-a886-c7baf9734bb2/31d43ba6-5b87-5475-9f10-ec280f14fb9b"
-					(reference "#PWR160")
+					(reference "#PWR161")
 					(unit 1)
 				)
@@
 		(on_board no)
 		(dnp no)
-		(property "Reference" "#PWR161"
+		(property "Reference" "#PWR162"
 			(at 168.91 180.34 0)
 			(effects
@@
 			(project "other-m68k"
 				(path "/0bd472a6-02e9-5c95-a886-c7baf9734bb2/31d43ba6-5b87-5475-9f10-ec280f14fb9b"
-					(reference "#PWR161")
-					(unit 1)
-				)
+					(reference "#PWR162")
+					(unit 1)
+				)
