File: kicad/release/other-m68k-power.kicad_sch (KiCad schematic)
At the start: 19 parts, among them J1 USB-C power, U12 AP2112K-3.3

Commit message: spec rev 11 / board rev C3: Atari joystick and paddle port on the DUART's I/O pins
Hardware: J12, a DE-9 male with the Atari pinout on the front edge. The five switches go
through 1 k into DUART inputs IP0..IP4 (up, down, left, right, fire), which already have
10 k pull-ups. Paddles: each pot charges, through 1 k, a 15 nF capacitor; a 74HC14 gate
(U14) pulls the up (A) or down (B) line low through a BAT54W when the capacitor passes its
threshold, so those lines double as end-of-charge signals (a joystick has no pots, paddles
no up/down switches); a dual NPN (Q1) on OP0 shorts both capacitors (pin high = shorted,
the reset state); +5 V through a 200 mA polyfuse. Paddle A's button is on pin 4 (right),
B's on pin 3 (left). The dedication moved under the SRAMs to make room. Routed with the
optimizer off: 0 DRC violations, 0 unrouted; fab package and release regenerated; the six
new part numbers are flagged verify in parts.json.

Firmware (fw/joy.c): sys_joystick (40) returns the JOY_* mask from one input-port read.
sys_paddles (41) fills struct paddles {a, b 0..1023 (1023 = 12 ms = 2764 counts), valid
bits, frame}: the first call starts measuring, NULL or program exit stops it. The
counter/timer runs free in timer mode from X1/16 (230.4 kHz) and IP0/IP1 change
interrupts are enabled (ACR 0x73, IMR.IPC). Each frame the VBLANK handler shorts the
capacitors; when the DUART reports the lines rising (its 38.4 kHz sampler has seen the
step) the level-3 handler releases them and notes the counter, and it timestamps each
fall; if nothing rose the next VBLANK releases directly. Measured in the emulator: 0.2 %
of the CPU with no paddle, 1.8 % with two. A joystick held up/down while measuring reads
as no paddle; a program using the counter/timer itself must not use paddles.

Spec: joystick section, DUART IPCR/ACR/IP/OPR fields, syscalls 40-41, struct paddles,
JOY_*/PADDLE_* constants. Emulator: joy.c models the port (--joy switches, --paddle A,B
or a game controller's triggers, SD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
Parts:
- removed C48: 100uF, Capacitor_THT:CP_Radial_D6.3mm_P2.50mm, symbol Device:C_Polarized
- removed C49: 10uF, Capacitor_SMD:C_0805_2012Metric, symbol Device:C
- removed C50: 1uF, Capacitor_SMD:C_0603_1608Metric, symbol Device:C
- removed R49, R50: 5.1k, Resistor_SMD:R_0603_1608Metric, symbol Device:R
- removed R51: 1k, Resistor_SMD:R_0603_1608Metric, symbol Device:R
- added C52: 10uF, Capacitor_SMD:C_0805_2012Metric, symbol Device:C
- added C53, C54: 1uF, Capacitor_SMD:C_0603_1608Metric, symbol Device:C
- added R58, R59: 5.1k, Resistor_SMD:R_0603_1608Metric, symbol Device:R
- added R60: 1k, Resistor_SMD:R_0603_1608Metric, symbol Device:R
- C51: value 1uF -> 100uF; footprint Capacitor_SMD:C_0603_1608Metric -> Capacitor_THT:CP_Radial_D6.3mm_P2.50mm; symbol Device:C -> Device:C_Polarized; Desc 1 uF 50 V X5R 0603 -> 100 uF 35 V electrolytic, 6.3 mm dia, 2.5 mm pitch (the 16 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; LCSC C15849 -> (none); MPN CL10A105KB8NNNC -> 35ZLH100MEFC6.3X11; Manufacturer Samsung -> Rubycon; PcbNear U12 -> J1
Connections:
- net +3V3: now also C54.1; no longer C51.1
- net CC1: now also R58.1
- net CC2: now also R59.1
- net GND: now also C52.2, C53.2, C54.2, R58.2, R59.2
- net PWRLED_A: now also R60.2
- net VCC: now also C51.1, C52.1, C53.1, R60.1
Changed lines of the file:
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@@
 		(on_board yes)
 		(dnp no)
-		(property "Reference" "C51"
+		(property "Reference" "C54"
 			(at 240.665 109.22 0)
 			(effects
@@
 			(project "other-m68k"
 				(path "/0bd472a6-02e9-5c95-a886-c7baf9734bb2/31d43ba6-5b87-5475-9f10-ec280f14fb9b"
-					(reference "C51")
+					(reference "C54")
 					(unit 1)
 				)
@@
 		(on_board yes)
 		(dnp no)
-		(property "Reference" "C50"
+		(property "Reference" "C53"
 			(at 175.895 109.22 0)
 			(effects
@@
 			(project "other-m68k"
 				(path "/0bd472a6-02e9-5c95-a886-c7baf9734bb2/31d43ba6-5b87-5475-9f10-ec280f14fb9b"
-					(reference "C50")
+					(reference "C53")
 					(unit 1)
 				)
@@
 		(on_board yes)
 		(dnp no)
-		(property "Reference" "R51"
+		(property "Reference" "R60"
 			(at 174.752 139.7 90)
 			(effects
@@
 			(project "other-m68k"
 				(path "/0bd472a6-02e9-5c95-a886-c7baf9734bb2/31d43ba6-5b87-5475-9f10-ec280f14fb9b"
-					(reference "R51")
+					(reference "R60")
 					(unit 1)
 				)
@@
 		(on_board yes)
 		(dnp no)
-		(property "Reference" "C49"
+		(property "Reference" "C52"
 			(at 112.395 109.22 0)
 			(effects
@@
 			(project "other-m68k"
 				(path "/0bd472a6-02e9-5c95-a886-c7baf9734bb2/31d43ba6-5b87-5475-9f10-ec280f14fb9b"
-					(reference "C49")
+					(reference "C52")
 					(unit 1)
 				)
@@
 		(on_board yes)
 		(dnp no)
-		(property "Reference" "C48"
+		(property "Reference" "C51"
 			(at 47.625 109.22 0)
 			(effects
@@
 			(project "other-m68k"
 				(path "/0bd472a6-02e9-5c95-a886-c7baf9734bb2/31d43ba6-5b87-5475-9f10-ec280f14fb9b"
-					(reference "C48")
+					(reference "C51")
 					(unit 1)
 				)
@@
 		(on_board yes)
 		(dnp no)
-		(property "Reference" "R50"
+		(property "Reference" "R59"
 			(at 111.252 139.7 90)
 			(effects
@@
 			(project "other-m68k"
 				(path "/0bd472a6-02e9-5c95-a886-c7baf9734bb2/31d43ba6-5b87-5475-9f10-ec280f14fb9b"
-					(reference "R50")
+					(reference "R59")
 					(unit 1)
 				)
@@
 		(on_board yes)
 		(dnp no)
-		(property "Reference" "R49"
+		(property "Reference" "R58"
 			(at 47.752 139.7 90)
 			(effects
@@
 			(project "other-m68k"
 				(path "/0bd472a6-02e9-5c95-a886-c7baf9734bb2/31d43ba6-5b87-5475-9f10-ec280f14fb9b"
-					(reference "R49")
+					(reference "R58")
 					(unit 1)
 				)
@@
 		(on_board no)
 		(dnp no)
-		(property "Reference" "#PWR143"
+		(property "Reference" "#PWR153"
 			(at 138.43 48.26 0)
 			(effects
@@
 			(project "other-m68k"
 				(path "/0bd472a6-02e9-5c95-a886-c7baf9734bb2/31d43ba6-5b87-5475-9f10-ec280f14fb9b"
-					(reference "#PWR143")
+					(reference "#PWR153")
 					(unit 1)
 				)
@@
 		(on_board no)
 		(dnp no)
-		(property "Reference" "#PWR144"
+		(property "Reference" "#PWR154"
 			(at 46.99 69.85 0)
 			(effects
@@
 			(project "other-m68k"
 				(path "/0bd472a6-02e9-5c95-a886-c7baf9734bb2/31d43ba6-5b87-5475-9f10-ec280f14fb9b"
-					(reference "#PWR144")
+					(reference "#PWR154")
 					(unit 1)
 				)
@@
 		(on_board no)
 		(dnp no)
-		(property "Reference" "#PWR145"
+		(property "Reference" "#PWR155"
 			(at 54.61 69.85 0)
 			(effects
@@
 			(project "other-m68k"
 				(path "/0bd472a6-02e9-5c95-a886-c7baf9734bb2/31d43ba6-5b87-5475-9f10-ec280f14fb9b"
-					(reference "#PWR145")
+					(reference "#PWR155")
 					(unit 1)
 				)
@@
 		(on_board no)
 		(dnp no)
-		(property "Reference" "#PWR146"
+		(property "Reference" "#PWR156"
 			(at 234.95 78.74 0)
 			(effects
@@
 			(project "other-m68k"
 				(path "/0bd472a6-02e9-5c95-a886-c7baf9734bb2/31d43ba6-5b87-5475-9f10-ec280f14fb9b"
-					(reference "#PWR146")
+					(reference "#PWR156")
 					(unit 1)
 				)
@@
 		(on_board no)
 		(dnp no)
-		(property "Reference" "#PWR147"
+		(property "Reference" "#PWR157"
 			(at 207.01 44.45 0)
 			(effects
@@
 			(project "other-m68k"
 				(path "/0bd472a6-02e9-5c95-a886-c7baf9734bb2/31d43ba6-5b87-5475-9f10-ec280f14fb9b"
-					(reference "#PWR147")
+					(reference "#PWR157")
 					(unit 1)
 				)
@@
 		(on_board no)
 		(dnp no)
-		(property "Reference" "#PWR148"
+		(property "Reference" "#PWR158"
 			(at 45.72 97.79 0)
 			(effects
@@
 			(project "other-m68k"
 				(path "/0bd472a6-02e9-5c95-a886-c7baf9734bb2/31d43ba6-5b87-5475-9f10-ec280f14fb9b"
-					(reference "#PWR148")
+					(reference "#PWR158")
 					(unit 1)
 				)
@@
 		(on_board no)
 		(dnp no)
-		(property "Reference" "#PWR149"
+		(property "Reference" "#PWR159"
 			(at 109.22 97.79 0)
 			(effects
@@
 			(project "other-m68k"
 				(path "/0bd472a6-02e9-5c95-a886-c7baf9734bb2/31d43ba6-5b87-5475-9f10-ec280f14fb9b"
-					(reference "#PWR149")
+					(reference "#PWR159")
 					(unit 1)
 				)
@@
 		(on_board no)
 		(dnp no)
-		(property "Reference" "#PWR150"
+		(property "Reference" "#PWR160"
 			(at 171.45 97.79 0)
 			(effects
@@
 			(project "other-m68k"
 				(path "/0bd472a6-02e9-5c95-a886-c7baf9734bb2/31d43ba6-5b87-5475-9f10-ec280f14fb9b"
-					(reference "#PWR150")
+					(reference "#PWR160")
 					(unit 1)
 				)
@@
 		(on_board no)
 		(dnp no)
-		(property "Reference" "#PWR151"
+		(property "Reference" "#PWR161"
 			(at 45.72 153.67 0)
 			(effects
@@
 			(project "other-m68k"
 				(path "/0bd472a6-02e9-5c95-a886-c7baf9734bb2/31d43ba6-5b87-5475-9f10-ec280f14fb9b"
-					(reference "#PWR151")
+					(reference "#PWR161")
 					(unit 1)
 				)
@@
 		(on_board no)
 		(dnp no)
-		(property "Reference" "#PWR152"
+		(property "Reference" "#PWR162"
 			(at 109.22 153.67 0)
 			(effects
@@
 			(project "other-m68k"
 				(path "/0bd472a6-02e9-5c95-a886-c7baf9734bb2/31d43ba6-5b87-5475-9f10-ec280f14fb9b"
-					(reference "#PWR152")
+					(reference "#PWR162")
 					(unit 1)
 				)
@@
 		(on_board no)
 		(dnp no)
-		(property "Reference" "#PWR153"
+		(property "Reference" "#PWR163"
 			(at 46.99 107.95 0)
 			(effects
@@
 			(project "other-m68k"
 				(path "/0bd472a6-02e9-5c95-a886-c7baf9734bb2/31d43ba6-5b87-5475-9f10-ec280f14fb9b"
-					(reference "#PWR153")
+					(reference "#PWR163")
 					(unit 1)
 				)
@@
 		(on_board no)
 		(dnp no)
-		(property "Reference" "#PWR154"
+		(property "Reference" "#PWR164"
 			(at 46.99 125.73 0)
 			(effects
@@
 			(project "other-m68k"
 				(path "/0bd472a6-02e9-5c95-a886-c7baf9734bb2/31d43ba6-5b87-5475-9f10-ec280f14fb9b"
-					(reference "#PWR154")
+					(reference "#PWR164")
 					(unit 1)
 				)
@@
 		(on_board no)
 		(dnp no)
-		(property "Reference" "#PWR155"
+		(property "Reference" "#PWR165"
 			(at 111.76 107.95 0)
 			(effects
@@
 			(project "other-m68k"
 				(path "/0bd472a6-02e9-5c95-a886-c7baf9734bb2/31d43ba6-5b87-5475-9f10-ec280f14fb9b"
-					(reference "#PWR155")
+					(reference "#PWR165")
 					(unit 1)
 				)
@@
 		(on_board no)
 		(dnp no)
-		(property "Reference" "#PWR156"
+		(property "Reference" "#PWR166"
 			(at 111.76 125.73 0)
 			(effects
@@
 			(project "other-m68k"
 				(path "/0bd472a6-02e9-5c95-a886-c7baf9734bb2/31d43ba6-5b87-5475-9f10-ec280f14fb9b"
-					(reference "#PWR156")
+					(reference "#PWR166")
 					(unit 1)
 				)
@@
 		(on_board no)
 		(dnp no)
-		(property "Reference" "#PWR157"
+		(property "Reference" "#PWR167"
 			(at 172.72 135.89 0)
 			(effects
@@
 			(project "other-m68k"
 				(path "/0bd472a6-02e9-5c95-a886-c7baf9734bb2/31d43ba6-5b87-5475-9f10-ec280f14fb9b"
-					(reference "#PWR157")
+					(reference "#PWR167")
 					(unit 1)
 				)
@@
 		(on_board no)
 		(dnp no)
-		(property "Reference" "#PWR158"
+		(property "Reference" "#PWR168"
 			(at 175.26 107.95 0)
 			(effects
@@
 			(project "other-m68k"
 				(path "/0bd472a6-02e9-5c95-a886-c7baf9734bb2/31d43ba6-5b87-5475-9f10-ec280f14fb9b"
-					(reference "#PWR158")
+					(reference "#PWR168")
 					(unit 1)
 				)
@@
 		(on_board no)
 		(dnp no)
-		(property "Reference" "#PWR159"
+		(property "Reference" "#PWR169"
 			(at 175.26 125.73 0)
 			(effects
@@
 			(project "other-m68k"
 				(path "/0bd472a6-02e9-5c95-a886-c7baf9734bb2/31d43ba6-5b87-5475-9f10-ec280f14fb9b"
-					(reference "#PWR159")
+					(reference "#PWR169")
 					(unit 1)
 				)
@@
 		(on_board no)
 		(dnp no)
-		(property "Reference" "#PWR160"
+		(property "Reference" "#PWR170"
 			(at 240.03 107.95 0)
 			(effects
@@
 			(project "other-m68k"
 				(path "/0bd472a6-02e9-5c95-a886-c7baf9734bb2/31d43ba6-5b87-5475-9f10-ec280f14fb9b"
-					(reference "#PWR160")
+					(reference "#PWR170")
 					(unit 1)
 				)
@@
 		(on_board no)
 		(dnp no)
-		(property "Reference" "#PWR161"
+		(property "Reference" "#PWR171"
 			(at 240.03 125.73 0)
 			(effects
@@
 			(project "other-m68k"
 				(path "/0bd472a6-02e9-5c95-a886-c7baf9734bb2/31d43ba6-5b87-5475-9f10-ec280f14fb9b"
-					(reference "#PWR161")
+					(reference "#PWR171")
 					(unit 1)
 				)
@@
 		(on_board no)
 		(dnp no)
-		(property "Reference" "#PWR162"
+		(property "Reference" "#PWR172"
 			(at 168.91 180.34 0)
 			(effects
@@
 			(project "other-m68k"
 				(path "/0bd472a6-02e9-5c95-a886-c7baf9734bb2/31d43ba6-5b87-5475-9f10-ec280f14fb9b"
-					(reference "#PWR162")
-					(unit 1)
-				)
+					(reference "#PWR172")
+					(unit 1)
+				)

Commit message: BOM: PCBWay descriptions carry only the part and its substitution rule; our sourcing remarks move to a Note field in parts.json, the KiCad BOM and the customer-parts list
Co-Authored-By: Claude Fable 5.1 <noreply@anthropic.com>
Claude-Session: https://claude.ai/code/session_019bbFLKMxhKXGW6aABP44Z1
Parts:
- C51: Desc 100 uF 35 V electrolytic, 6.3 mm dia, 2.5 mm pitch (the 16 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 -> 100 uF 35 V electrolytic, 6.3 mm dia, 2.5 mm pitch; Note (none) -> 35 V part chosen for the can size: the 16 V ZLH 100 uF is a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
- J1: Desc USB-C receptacle, 6 pin, power only, right angle (DigiKey/F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 -> USB-C receptacle, 6 pin, power only, right angle; Note (none) -> DigiKey/Farnell/Future list it; stock varies
Changed lines of the file:
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@@
 			)
 		)
-		(property "Desc" "100 uF 35 V electrolytic, 6.3 mm dia, 2.5 mm pitch (the 16 V ZLH 100 uF is a 5 mm can)"
+		(property "Desc" "100 uF 35 V electrolytic, 6.3 mm dia, 2.5 mm pitch"
+			(at 46.99 111.76 0)
+			(effects
+				(font
+					(size 1.27 1.27)
+				)
+				(hide yes)
+			)
+		)
+		(property "Note" "35 V part chosen for the can size: the 16 V ZLH 100 uF is a 5 mm can"
 			(at 46.99 111.76 0)
 			(effects
@@
 			)
 		)
-		(property "Desc" "USB-C receptacle, 6 pin, power only, right angle (DigiKey/Farnell/Future list it; stock varies)"
+		(property "Desc" "USB-C receptacle, 6 pin, power only, right angle"
 			(at 54.61 41.91 0)
 			(effects
+				(font
+					(size 1.27 1.27)
+				)
+				(hide yes)
+			)
+		)
+		(property "Note" "DigiKey/Farnell/Future list it; stock varies"
+			(at 54.61 41.91 0)
+			(effects
