File: kicad/release/other-m68k-cpld1.kicad_sch (KiCad schematic)
At the start: 15 parts, among them J7 JTAG (ByteBlaster), U6 ATF1508AS-7JX84 (MMU), X1 24MHz

Commit message: rev C3 BOM: in-stock substitutes from the PCBWay quote: ECS-2200B-240 oscillator, Assmann PLCC-84 and DIP-40 sockets, generic DIP-64 socket acceptable
Co-Authored-By: Claude Fable 5.1 <noreply@anthropic.com>
Claude-Session: https://claude.ai/code/session_019bbFLKMxhKXGW6aABP44Z1
Parts:
- U6: Socket_Desc PLCC-84 through-hole socket, 1.27 mm pitch (RS 7019411) -> PLCC-84 through-hole socket, 1.27 mm pitch (DigiKey 5023770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; Socket_MPN 540-88-084-24-008 -> A-CCS-084-Z-T; Socket_Manufacturer Preci-dip -> Assmann WSW
- X1: Desc 24 MHz 5 V HCMOS oscillator, half-size DIP-8 (DigiKey: 18 w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 -> 24 MHz 5 V HCMOS oscillator, half-size DIP-8 with tri-state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; MPN ECS-2100A-240 -> ECS-2200B-240
Changed lines of the file:
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@@
 			)
 		)
-		(property "MPN" "ECS-2100A-240"
+		(property "MPN" "ECS-2200B-240"
 			(at 154.94 33.02 0)
 			(effects
@@
 			)
 		)
-		(property "Desc" "24 MHz 5 V HCMOS oscillator, half-size DIP-8 (DigiKey: 18 week lead time 2026-10; any 5 V half-size DIP-8 oscillator fits)"
+		(property "Desc" "24 MHz 5 V HCMOS oscillator, half-size DIP-8 with tri-state pin 1 (internal pull-up, tied to VCC here; DigiKey in stock 2026-10; the ECS-2100A-240 is 18 weeks). Any 5 V half-size DIP-8 oscillator fits"
 			(at 154.94 33.02 0)
 			(effects
@@
 			)
 		)
-		(property "Socket_Manufacturer" "Preci-dip"
+		(property "Socket_Manufacturer" "Assmann WSW"
 			(at 62.23 76.2 0)
 			(effects
@@
 			)
 		)
-		(property "Socket_MPN" "540-88-084-24-008"
+		(property "Socket_MPN" "A-CCS-084-Z-T"
 			(at 62.23 76.2 0)
 			(effects
@@
 			)
 		)
-		(property "Socket_Desc" "PLCC-84 through-hole socket, 1.27 mm pitch (RS 7019411)"
+		(property "Socket_Desc" "PLCC-84 through-hole socket, 1.27 mm pitch (DigiKey 5023770 / AE11110-ND, RS 674-2555; any THT PLCC-84 socket with the JEDEC pin pattern is acceptable)"
 			(at 62.23 76.2 0)
 			(effects

Commit message: BOM: PCBWay descriptions carry only the part and its substitution rule; our sourcing remarks move to a Note field in parts.json, the KiCad BOM and the customer-parts list
Co-Authored-By: Claude Fable 5.1 <noreply@anthropic.com>
Claude-Session: https://claude.ai/code/session_019bbFLKMxhKXGW6aABP44Z1
Parts:
- U6: Socket_Desc PLCC-84 through-hole socket, 1.27 mm pitch (DigiKey 5023770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 -> PLCC-84 through-hole socket, 1.27 mm pitch; any THT PLCC-84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; Socket_Note (none) -> DigiKey 5023770 / AE11110-ND, RS 674-2555. Replaces the Pre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
- X1: Desc 24 MHz 5 V HCMOS oscillator, half-size DIP-8 with tri-state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 -> 24 MHz 5 V HCMOS oscillator, half-size DIP-8; any 5 V half-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; Note (none) -> ECS-2200B-240 has a tri-state pin 1 with internal pull-up; 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
Changed lines of the file:
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@@
 			)
 		)
-		(property "Desc" "24 MHz 5 V HCMOS oscillator, half-size DIP-8 with tri-state pin 1 (internal pull-up, tied to VCC here; DigiKey in stock 2026-10; the ECS-2100A-240 is 18 weeks). Any 5 V half-size DIP-8 oscillator fits"
+		(property "Desc" "24 MHz 5 V HCMOS oscillator, half-size DIP-8; any 5 V half-size DIP-8 oscillator whose pin 1 is NC or an active-high output enable fits (pin 1 is tied to VCC)"
+			(at 154.94 33.02 0)
+			(effects
+				(font
+					(size 1.27 1.27)
+				)
+				(hide yes)
+			)
+		)
+		(property "Note" "ECS-2200B-240 has a tri-state pin 1 with internal pull-up; DigiKey in stock 2026-10. The ECS-2100A-240 of the B4 BOM was 18 weeks"
 			(at 154.94 33.02 0)
 			(effects
@@
 			)
 		)
-		(property "Socket_Desc" "PLCC-84 through-hole socket, 1.27 mm pitch (DigiKey 5023770 / AE11110-ND, RS 674-2555; any THT PLCC-84 socket with the JEDEC pin pattern is acceptable)"
+		(property "Socket_Desc" "PLCC-84 through-hole socket, 1.27 mm pitch; any THT PLCC-84 socket with the JEDEC pin pattern is acceptable"
 			(at 62.23 76.2 0)
 			(effects
+				(font
+					(size 1.27 1.27)
+				)
+				(hide yes)
+			)
+		)
+		(property "Socket_Note" "DigiKey 5023770 / AE11110-ND, RS 674-2555. Replaces the Preci-dip PCBWay could not source (2026-10)"
+			(at 62.23 76.2 0)
+			(effects

Commit message: PCBWay BOM: the DIP-64 socket row asks for any 0.9 in dual-wipe socket with the Mill-Max as fallback, the oscillator row drops the pin 1 explanation; ORDER.md carries the short order-form remark instead of the bullet list
Co-Authored-By: Claude Fable 5.1 <noreply@anthropic.com>
Claude-Session: https://claude.ai/code/session_019bbFLKMxhKXGW6aABP44Z1
Parts:
- X1: Desc 24 MHz 5 V HCMOS oscillator, half-size DIP-8; any 5 V half-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 -> 24 MHz 5 V HCMOS oscillator, half-size DIP-8; any 24 MHz 5 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; Note ECS-2200B-240 has a tri-state pin 1 with internal pull-up; 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 -> Pin 1 is tied to VCC, so any part with pin 1 NC or an activ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
Changed lines of the file:
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@@
 			)
 		)
-		(property "Desc" "24 MHz 5 V HCMOS oscillator, half-size DIP-8; any 5 V half-size DIP-8 oscillator whose pin 1 is NC or an active-high output enable fits (pin 1 is tied to VCC)"
+		(property "Desc" "24 MHz 5 V HCMOS oscillator, half-size DIP-8; any 24 MHz 5 V half-size DIP-8 oscillator is acceptable"
 			(at 154.94 33.02 0)
 			(effects
@@
 			)
 		)
-		(property "Note" "ECS-2200B-240 has a tri-state pin 1 with internal pull-up; DigiKey in stock 2026-10. The ECS-2100A-240 of the B4 BOM was 18 weeks"
+		(property "Note" "Pin 1 is tied to VCC, so any part with pin 1 NC or an active-high enable fits; the ECS-2200B-240 has a tri-state pin 1 with internal pull-up. DigiKey in stock 2026-10; the ECS-2100A-240 of the B4 BOM was 18 weeks"
 			(at 154.94 33.02 0)
 			(effects
