File: kicad/release/other-m68k-cpu.kicad_sch (KiCad schematic)
At the start: 18 parts, among them J9 Logic analyzer (gusmanb 2x15), U1 MC68000P12

Commit message: rev C3 BOM: in-stock substitutes from the PCBWay quote: ECS-2200B-240 oscillator, Assmann PLCC-84 and DIP-40 sockets, generic DIP-64 socket acceptable
Co-Authored-By: Claude Fable 5.1 <noreply@anthropic.com>
Claude-Session: https://claude.ai/code/session_019bbFLKMxhKXGW6aABP44Z1
Parts:
- U1: Socket_Desc DIP-64 socket, 22.86 mm (0.9 in) rows, gold contacts, RoHS -> DIP-64 socket, 22.86 mm (0.9 in) rows. ANY dual-wipe (stamp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
Changed lines of the file:
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@@
 			)
 		)
-		(property "Socket_Desc" "DIP-64 socket, 22.86 mm (0.9 in) rows, gold contacts, RoHS"
+		(property "Socket_Desc" "DIP-64 socket, 22.86 mm (0.9 in) rows. ANY dual-wipe (stamped tin) DIP-64 socket with 0.9 in row spacing is acceptable and preferred on cost; the Mill-Max machined part is the fallback (PCBWay quoted it at $38, DigiKey sells it for about $15, so consigning it is an option)"
 			(at 59.69 100.33 0)
 			(effects

Commit message: BOM: PCBWay descriptions carry only the part and its substitution rule; our sourcing remarks move to a Note field in parts.json, the KiCad BOM and the customer-parts list
Co-Authored-By: Claude Fable 5.1 <noreply@anthropic.com>
Claude-Session: https://claude.ai/code/session_019bbFLKMxhKXGW6aABP44Z1
Parts:
- U1: Socket_Desc DIP-64 socket, 22.86 mm (0.9 in) rows. ANY dual-wipe (stamp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 -> DIP-64 socket, 22.86 mm (0.9 in) rows; any dual-wipe (stamp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; Socket_Note (none) -> PCBWay quoted the Mill-Max at $38 (2026-10); DigiKey sells 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
Changed lines of the file:
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@@
 			)
 		)
-		(property "Socket_Desc" "DIP-64 socket, 22.86 mm (0.9 in) rows. ANY dual-wipe (stamped tin) DIP-64 socket with 0.9 in row spacing is acceptable and preferred on cost; the Mill-Max machined part is the fallback (PCBWay quoted it at $38, DigiKey sells it for about $15, so consigning it is an option)"
+		(property "Socket_Desc" "DIP-64 socket, 22.86 mm (0.9 in) rows; any dual-wipe (stamped tin) DIP-64 socket with 0.9 in row spacing is acceptable and preferred, this machined part is the fallback"
 			(at 59.69 100.33 0)
 			(effects
+				(font
+					(size 1.27 1.27)
+				)
+				(hide yes)
+			)
+		)
+		(property "Socket_Note" "PCBWay quoted the Mill-Max at $38 (2026-10); DigiKey sells it for about $15. No stamped 0.9 in DIP-64 found at DigiKey/Mouser"
+			(at 59.69 100.33 0)
+			(effects

Commit message: PCBWay BOM: the DIP-64 socket row asks for any 0.9 in dual-wipe socket with the Mill-Max as fallback, the oscillator row drops the pin 1 explanation; ORDER.md carries the short order-form remark instead of the bullet list
Co-Authored-By: Claude Fable 5.1 <noreply@anthropic.com>
Claude-Session: https://claude.ai/code/session_019bbFLKMxhKXGW6aABP44Z1
Parts:
- U1: Socket_Desc DIP-64 socket, 22.86 mm (0.9 in) rows; any dual-wipe (stamp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 -> DIP-64 socket, 22.86 mm (0.9 in) row spacing, stamped dual-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; Socket_MPN 110-43-964-41-001000 -> DIP-64 socket, 0.9 in rows, dual-wipe; Socket_Manufacturer Mill-Max -> any; Socket_Note PCBWay quoted the Mill-Max at $38 (2026-10); DigiKey sells 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 -> Named generically so the assembler looks for a stamped sock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
Changed lines of the file:
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@@
 			)
 		)
-		(property "Socket_Manufacturer" "Mill-Max"
+		(property "Socket_Manufacturer" "any"
 			(at 59.69 100.33 0)
 			(effects
@@
 			)
 		)
-		(property "Socket_MPN" "110-43-964-41-001000"
+		(property "Socket_MPN" "DIP-64 socket, 0.9 in rows, dual-wipe"
 			(at 59.69 100.33 0)
 			(effects
@@
 			)
 		)
-		(property "Socket_Desc" "DIP-64 socket, 22.86 mm (0.9 in) rows; any dual-wipe (stamped tin) DIP-64 socket with 0.9 in row spacing is acceptable and preferred, this machined part is the fallback"
+		(property "Socket_Desc" "DIP-64 socket, 22.86 mm (0.9 in) row spacing, stamped dual-wipe tin contacts; fallback if none is available: Mill-Max 110-43-964-41-001000 (machined)"
 			(at 59.69 100.33 0)
 			(effects
@@
 			)
 		)
-		(property "Socket_Note" "PCBWay quoted the Mill-Max at $38 (2026-10); DigiKey sells it for about $15. No stamped 0.9 in DIP-64 found at DigiKey/Mouser"
+		(property "Socket_Note" "Named generically so the assembler looks for a stamped socket first. PCBWay quoted the Mill-Max at $38 (2026-10); DigiKey sells it for about $15. No stamped 0.9 in DIP-64 found at DigiKey/Mouser"
 			(at 59.69 100.33 0)
 			(effects
