File: kicad/release/other-m68k.kicad_pcb (KiCad board)
At the start: 4 copper layers, 180 x 125 mm, 171 parts, among them J1 USB-C power, J10 S-video, J11 FTDI B (GND CTS VCC TXD RXD R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, J12 Joystick (Atari DE-9), J2 FTDI (GND CTS VCC TXD RXD RTS), J3 PS/2, J4 microSD DM3AT-SF-PEJM5, J5 RCA composite, J6 3.5mm audio, J7 JTAG (ByteBlaster), J9 Logic analyzer (gusmanb 2x15), Q1 MMDT3904, SW1 RESET, SW2 NMI, U1 MC68000P12, U10 MC68681P, U11 AD724JR, U12 AP2112K-3.3, U13 MCP130T-450I/TT, U14 74HC14, U2 AS6C4008-55PCN (upper, D15..D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, U3 AS6C4008-55PCN (lower, D7..D0), U4 SST39SF040-70 (even, D15..D8), U5 SST39SF040-70 (odd, D7..D0), U6 ATF1508AS-7JX84 (MMU), U7 ATF1508AS-7JX84 (I/O), U8 74AHCT245 (hi), U9 74AHCT245 (lo), X1 24MHz, Y1 3.6864MHz, Y2 3.579545MHz

Commit message: rev C3 silkscreen: drop the third dedication line, revision text reads "rev C3"
Edited in placement.json and directly in the routed board (text only, no reroute); DRC 0.

Co-Authored-By: Claude Fable 5.1 <noreply@anthropic.com>
Claude-Session: https://claude.ai/code/session_019bbFLKMxhKXGW6aABP44Z1
Other:
- board text added: "rev C3"
- board text removed: "I love you, Kris!"
- board text removed: "other-m68k rev C3"
Changed lines of the file:
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@@
 		)
 	)
-	(gr_text "other-m68k rev C3"
+	(gr_text "rev C3"
 		(at 162 43.4 0)
 		(layer "F.SilkS")
@@
 		(layer "F.SilkS")
 		(effects
-			(font
-				(size 1.7 1.7)
-				(thickness 0.255)
-			)
-		)
-	)
-	(gr_text "I love you, Kris!"
-		(at 162 55.6 0)
-		(layer "F.SilkS")
-		(effects

Commit message: rev C3 silkscreen: ODD and EVEN under the flash sockets U5 and U4
Text only, placed in the 1.5 mm strip between the socket outlines and the LED
reference designators (size 1.2 mm); edited in placement.json and the routed board, DRC 0.

Co-Authored-By: Claude Fable 5.1 <noreply@anthropic.com>
Claude-Session: https://claude.ai/code/session_019bbFLKMxhKXGW6aABP44Z1
Other:
- board text added: "EVEN"
- board text added: "ODD"
Changed lines of the file:
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@@
+		)
+	)
+	(gr_text "ODD"
+		(at 152.5 105.3 0)
+		(layer "F.SilkS")
+		(effects
+			(font
+				(size 1.2 1.2)
+				(thickness 0.18)
+			)
+		)
+	)
+	(gr_text "EVEN"
+		(at 169 105.3 0)
+		(layer "F.SilkS")
+		(effects
+			(font
+				(size 1.2 1.2)
+				(thickness 0.18)
+			)
 		)
 	)
